Commit message: plus imu to robot

File: src/f1_robot_model/urdf/racecar.urdf (robot description, URDF)
Before this commit: robot racecar, 9 links, 8 joints
Links:
- added link imu; collision box size=0.1 0.1 0.1; visual box size=0.01 0.01 0.01
- added link laser; collision box size=0.1 0.1 0.1; visual mesh filename=file://$(find f1_robot_model)/meshes/hokuyo.dae
Joints:
- added joint hokuyo_joint: type fixed, parent base_link, child laser, origin xyz=0.1 0.0 0.075 rpy=0 0 0, axis 0 0 1
- added joint imu_joint: type fixed, parent base_link, child imu, origin xyz=0.1 0.0 0.025 rpy=0.0 0.0 0.0, axis 0.0 0.0 1.0

Commit message: Add GPS and Fix README.md and CHANGELOG.md

File: src/f1_robot_model/urdf/racecar.urdf (robot description, URDF)
Before this commit: robot racecar, 11 links, 10 joints
Links:
- added link gps; collision box size=0.1 0.1 0.1; visual box size=0.01 0.01 0.01
Joints:
- added joint gps_joint: type fixed, parent base_link, child gps, origin xyz=0.1 0.0 0.03 rpy=0.0 0.0 0.0, axis 0.0 0.0 1.0
